Commit message: added commented 3D velodyne in accessories.urdf

File: spot_description/urdf/accessories.urdf.xacro (robot description, xacro)
@@ -4,4 +4,5 @@
     <xacro:include filename="$(find hector_sensors_description)/urdf/hokuyo_utm30lx.urdf.xacro" />
     <xacro:include filename="$(find hector_sensors_description)/urdf/asus_camera.urdf.xacro" />
+    <xacro:include filename="$(find velodyne_description)/urdf/VLP-16.urdf.xacro" />
     <xacro:hokuyo_utm30lx
         name="hokuyo"
@@ -14,4 +15,7 @@
         <origin xyz="0.0 0.0 ${base_height / 2 + 0.04}" rpy="0 0 0"/>
     </xacro:hokuyo_utm30lx>
+    <!--<xacro:VLP-16 parent="base_link" name="velodyne" topic="/velodyne_points" organize_cloud="True" hz="10" samples="440" gpu="True">
+    <origin xyz="0.0 0.0 ${base_height / 2 + 0.04}" rpy="0 0 0" />
+    </xacro:VLP-16>-->
     <gazebo reference="hokuyo_frame">
 		<material>Gazebo/FlatBlack</material>
